Commit message: :thought_balloon: Driver robot

File: description/robot.urdf.xacro (robot description, xacro)
@@ -5,4 +5,6 @@
     como se fosse uma lincagem pra main em C
      -->
-    <xacro:include filename="robot_core.xacro" />
+    <xacro:include filename="robot_core.xacro"/>
+    <!--Incluindo novo arquivo para controlar o robo no gazebo -->
+    <xacro:include filename="gazebo_control.xacro"/>
 </robot>

File: description/robot_core.xacro (robot description, xacro)
@@ -48,4 +48,8 @@
         </xacro:inertial_box>
     </link>
+    <!--Adicionando cores para o gazebo-->
+    <gazebo reference="chassis">
+        <material>Gazebo/Yellow</material>
+    </gazebo>
     <!-- ===================== LEFT WHEEL LINK ===================== -->
     <joint name="left_wheel_joint" type="continuous">
@@ -72,4 +76,7 @@
         </xacro:inertial_cylinder>
     </link>
+    <gazebo reference="left_wheel">
+        <material>Gazebo/Blue</material>
+    </gazebo>
     <!-- ===================== RIGHT WHEEL LINK ===================== -->
     <joint name="right_wheel_joint" type="continuous">
@@ -96,4 +103,7 @@
         </xacro:inertial_sphere>
     </link>
+    <gazebo reference="right_wheel">
+        <material>Gazebo/Blue</material>
+    </gazebo>
     <!-- ===================== CASTER WHEEL LINK ===================== -->
     <joint name="caster_wheel_joint" type="fixed">
@@ -119,3 +129,9 @@
         </xacro:inertial_sphere>
     </link>
+    <gazebo reference="caster_wheel">
+        <material>Gazebo/Red</material>
+        <!--(Reduzindo o atrito) para que a esfera possa girar -->
+        <mu1 value="0.001"/>
+        <mu2 value="0.001"/>
+    </gazebo>
 </robot>
